File: hardware/boards/glasgow/glasgow.sch (KiCad schematic (older format))
At the start: 93 parts, among them J1 USB_B_Micro, U1 CY7C68013A-56LTX, U15 TPD3S014, U2 CAT24M01W, U3 CAT24C256W, U30 ICE40HX8K-BG121, U34 ATECC508A, U36 TLV73312PQDRVRQ1, U7 LM3880MF-1AF, U8 TLV75533PDRVR, Y1 24M

Commit message: Revert "hardware/boards/glasgow: explain the function of R40."
This reverts commit e1c8c857491b0fe7a51a297b86bf74c5d51f8d3e.
Other:
- note removed: "Plug in the device while shorting R40 if it stops enumerating"
Changed lines of the file:
@@
-EESchema Schematic File Version 5
-EELAYER 30 0
+EESchema Schematic File Version 4
+LIBS:glasgow-cache
+EELAYER 29 0
 EELAYER END
 $Descr A4 11693 8268
@@
 Comment3 ""
 Comment4 ""
-Comment5 ""
-Comment6 ""
-Comment7 ""
-Comment8 ""
-Comment9 ""
 $EndDescr
 $Comp
@@
 Wire Wire Line
 	2300 3700 2300 4150
-Wire Notes Line
-	5300 7050 5300 7650
-Text Notes 4550 7750 0    50   ~ 0
-Plug in the device while shorting R40 if it stops enumerating
 Wire Bus Line
 	4700 6250 7850 6250

Commit message: Update schematic to use USB-C
In a misguided attempt to minimize
the amount of cables laying around
I decided that USB-C is the answer.
Parts:
- removed J1: USB_B_Micro, Connector_USB:USB_Micro-B_Molex_47346-0001, symbol Connector:USB_B_Micro
- added J1: USB_C_Receptacle_USB2.0, Connector_USB_git:USB_C_Receptacle_HRO_TYPE-C-31-M-12, symbol Connector:USB_C_Receptacle_USB2.0
- added R52, R53: 5k1, Resistor_SMD:R_0402_1005Metric, symbol Device:R
- U30: symbol FPGA_Lattice:ICE40HX8K-BG121 -> glasgow-rescue:ICE40HX8K-BG121-FPGA_Lattice
Connections:
- net GND: now also J1.A1 (GND), J1.A12 (GND), J1.B1 (GND), J1.B12 (GND), R52.2, R53.2
- net SHLD: now also J1.S1 (SHIELD)
- net USB_N: now also J1.A7 (D-), J1.B7 (D-)
- net USB_P: now also J1.A6 (D+), J1.B6 (D+)
- net at FB1.1, TP13.1: now also J1.A4 (VBUS), J1.A9 (VBUS), J1.B4 (VBUS), J1.B9 (VBUS)
- new net: J1.A5 (CC1), R52.1
- new net: J1.B5 (CC2), R53.1
- no-connect marks 8 -> 9
Other:
- moved on the sheet: C13, FB1, MK1, MK2, MK3, MK4, R3, TP13, TP14, TP15, TP16
