File: hardware/boards/glasgow/io_banks.sch (KiCad schematic (older format))
At the start: 26 parts, among them J10 Conn_01x03, J4 Conn_01x02, J5 Conn_02x22_Odd_Even, U30 ICE40HX8K-BG121, U32 SN74LVC1T45DRL

Commit message: Update schematic to use USB-C
In a misguided attempt to minimize
the amount of cables laying around
I decided that USB-C is the answer.
Parts:
- U30: symbol FPGA_Lattice:ICE40HX8K-BG121 -> glasgow-rescue:ICE40HX8K-BG121-FPGA_Lattice
Changed lines of the file:
@@
 	1300 2850 1300 2800
 $Comp
-L FPGA_Lattice:ICE40HX8K-BG121 U?
+L glasgow-rescue:ICE40HX8K-BG121-FPGA_Lattice U?
 U 2 1 5C9E33E2
 P 4750 4450
@@
 $EndComp
 $Comp
-L FPGA_Lattice:ICE40HX8K-BG121 U?
+L glasgow-rescue:ICE40HX8K-BG121-FPGA_Lattice U?
 U 4 1 5C9E33E9
 P 8250 4200
@@
 $EndComp
 $Comp
-L FPGA_Lattice:ICE40HX8K-BG121 U?
+L glasgow-rescue:ICE40HX8K-BG121-FPGA_Lattice U?
 U 1 1 5C9E33DB
 P 1300 4250
